File: Hrbl_for_shopbot/KiCAD_files/nano.sch (KiCad schematic (older format))
At the start: 69 parts, among them P1 Digital, P2 Analog, P3 CONN_01X01, P4 CONN_01X01, P5 CONN_01X01, P6 CONN_01X01, U1 SFH6206-3T, U10 SFH6206-3T, U11 SFH6206-3T, U12 SFH6206-3T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

Commit message: Updated with 24V Contactor signal and PWM filter
Parts:
- added POWER_IN2: Conn_01x02, Connector_Phoenix_MC:PhoenixContact_MCV_1,5_2-G-3.5_1x02_P3.50mm_Vertical, symbol Connector_Generic:Conn_01x02
- added R27: R 1k, Resistor_SMD:R_1206_3216Metric_Pad1.42x1.75mm_HandSolder, symbol Device:R
- C4: value 100nF (0.1uF) -> 10uF
- R12: value 220 -> R 1k
Connections:
- net 5V_ISO: no longer R12.2
- net GNDS: now also POWER_IN2.2 (Pin_2)
- net VI: now also R27.2; no longer C4.1, SPINDLE1.3 (Pin_3)
- new net: C4.1, R27.1, SPINDLE1.3 (Pin_3)
- new net 24V_CONTACTOR_SIGNAL: POWER_IN2.1 (Pin_1), R12.2
Other:
- note added: "Abort indicator, on the front!"
- note removed: "Abort indicator"
Changed lines of the file:
@@
 P 5350 2100
 F 0 "R12" H 5300 2100 50  0000 L CNN
-F 1 "220" H 5150 2050 50  0000 L CNN
+F 1 "R 1k" H 5100 2100 50  0000 L CNN
 F 2 "Resistor_SMD:R_1206_3216Metric_Pad1.42x1.75mm_HandSolder" V 5280 2100 50  0001 C CNN
 F 3 "~" H 5350 2100 50  0001 C CNN
@@
 $EndComp
 Text GLabel 5200 2100 0    50   Input ~ 0
-5V_ISO
+24V_CONTACTOR_SIGNAL
 $Comp
 L power:GNDS #PWR07
@@
 	7300 1950 7300 2100
 Text Notes 7600 1800 0    50   ~ 0
-Abort indicator
+Abort indicator, on the front!
 Text Notes 7150 2600 0    50   ~ 0
 Arduino GND!
@@
 P 12250 6850
 F 0 "C4" H 12428 6896 50  0000 L CNN
-F 1 "100nF (0.1uF)" H 12428 6805 50  0000 L CNN
+F 1 "10uF" H 12428 6805 50  0000 L CNN
 F 2 "Capacitor_SMD:C_1206_3216Metric_Pad1.42x1.75mm_HandSolder" H 12250 6850 50  0001 C CNN
 F 3 "" H 12250 6850 50  0001 C CNN
@@
 	12550 7100 12250 7100
 Wire Wire Line
-	12250 6600 11900 6600
-Wire Wire Line
-	11900 6600 11900 6950
-Wire Wire Line
 	11900 6950 11350 6950
-Connection ~ 12250 6600
 Wire Wire Line
 	12250 7100 11850 7100
@@
 	1    0    0    -1
 $EndComp
+$Comp
+L Connector_Generic:Conn_01x02 POWER_IN2
+U 1 1 5BC54375
+P 14100 8450
+F 0 "POWER_IN2" H 14180 8442 50  0000 L CNN
+F 1 "Conn_01x02" H 14180 8351 50  0000 L CNN
+F 2 "Connector_Phoenix_MC:PhoenixContact_MCV_1,5_2-G-3.5_1x02_P3.50mm_Vertical" H 14100 8450 50  0001 C CNN
+F 3 "~" H 14100 8450 50  0001 C CNN
+	1    14100 8450
+	1    0    0    -1
+$EndComp
+Text GLabel 13600 8450 0    50   Input ~ 0
+24V_CONTACTOR_SIGNAL
+$Comp
+L power:GNDS #PWR038
+U 1 1 5BC564F4
+P 13600 8550
+F 0 "#PWR038" H 13600 8300 50  0001 C CNN
+F 1 "GNDS" V 13605 8422 50  0000 R CNN
+F 2 "" H 13600 8550 50  0001 C CNN
+F 3 "" H 13600 8550 50  0001 C CNN
+	1    13600 8550
+	0    1    1    0
+$EndComp
+Wire Wire Line
+	13600 8450 13900 8450
+Wire Wire Line
+	13900 8550 13600 8550
+$Comp
+L Device:R R27
+U 1 1 5BC6D809
+P 12100 6600
+F 0 "R27" V 11893 6600 50  0000 C CNN
+F 1 "R 1k" V 11984 6600 50  0000 C CNN
+F 2 "Resistor_SMD:R_1206_3216Metric_Pad1.42x1.75mm_HandSolder" V 12030 6600 50  0001 C CNN
+F 3 "~" H 12100 6600 50  0001 C CNN
+	1    12100 6600
+	0    1    1    0
+$EndComp
+Connection ~ 12250 6600
+Wire Wire Line
+	11950 6600 11900 6600
+Wire Wire Line
+	11900 6600 11900 6950
 $EndSCHEMATC

Commit message: Kicad files
Parts:
- removed P3, P4, P5, P6: CONN_01X01, Socket_Arduino_Nano:1pin_Nano, symbol Connector_Generic:Conn_01x01
- removed R11: 220, Resistor_SMD:R_1206_3216Metric_Pad1.42x1.75mm_HandSolder, symbol Device:R
- removed R27: R 1k, Resistor_SMD:R_1206_3216Metric_Pad1.42x1.75mm_HandSolder, symbol Device:R
- removed SPINDLE1: Conn_01x04, Connector_Phoenix_MC:PhoenixContact_MCV_1,5_4-G-3.5_1x04_P3.50mm_Vertical, symbol Connector_Generic:Conn_01x04
- removed U3: SFH6206-3T, Package_DIP:SMDIP-4_W9.53mm_Clearance8mm, symbol Isolator:SFH6206-3T
- added C?: 10uF, Capacitor_SMD:C_1206_3216Metric_Pad1.42x1.75mm_HandSolder, symbol pspice:CAP
- added R?: 220, Resistor_SMD:R_1206_3216Metric_Pad1.42x1.75mm_HandSolder, symbol Device:R
- added R?: R 680, Resistor_SMD:R_1206_3216Metric_Pad1.42x1.75mm_HandSolder, symbol Device:R
- added R?: R 220, Resistor_SMD:R_1206_3216Metric_Pad1.42x1.75mm_HandSolder, symbol Device:R
- added SPID_EN: Conn_01x02, Connector_Phoenix_MC:PhoenixContact_MCV_1,5_2-G-3.5_1x02_P3.50mm_Vertical, symbol Connector_Generic:Conn_01x02
- added SPIN_PWM: Conn_01x04, Connector_Phoenix_MC:PhoenixContact_MCV_1,5_4-G-3.5_1x04_P3.50mm_Vertical, symbol Connector_Generic:Conn_01x04
- added U? (x2): SFH6206-3T, Package_DIP:SMDIP-4_W9.53mm_Clearance8mm, symbol Isolator:SFH6206-3T
Connections:
- net +5V: now also R?.2
- net 5V_ISO: no longer U7.4
- net A1: now also C4.1, C?.1, R?.2, SPIN_PWM.2 (Pin_2)
- net ALARM_IN: now also U?.3
- net GND: no longer U7.2
- net GNDS: no longer C4.2
- net SPINDLE_PWM: now also U7.2
- net at U7.1: now also R?.1
- net at R13.1: now also U?.4
- net DCM(COM) renamed SC
- net SC: now also SPID_EN.2 (Pin_2)
- net FOR renamed S1
- net S1: now also SPID_EN.1 (Pin_1)
- net VI renamed AC
- net AC: now also C4.2, C?.2, SPIN_PWM.3 (Pin_3)
- new net: R?.1, R?.1, U7.4
- new net V+: R?.2, SPIN_PWM.1 (Pin_1)
- no-connect marks 16 -> 13
Other:
- note added: "+24V in SOURCE SPINDLE FOR"
- note added: "A1 (20k)"
- note added: "AC"
- note added: "All motors ALARM in SERIES!! -> IN HERE\n"
- note added: "S1"
- note added: "SC"
- note added: "SINK 17mA"
- note added: "SOURCE 17mA"
- note added: "TOT SOURCE 119mA"
- note added: "V+ (10.5V)\n"
- note added: "VFD GND"
- note added: "alarm in HIGH = No alarm\nMAKE INVERTER AS FOR CONNECTOR\n"
- note added: "second contactor"
- note removed: "+24V in"
- note removed: "ACM(GND)"
- note removed: "All motors ALARM in Parallell"
- note removed: "DCM(COM)"
- note removed: "FOR"
- note removed: "Holes"
- note removed: "Spindle_EN_out"
- note removed: "VI\n"
- moved on the sheet: C1, C2, C3, C4, C5, C6, MH1, MH2, MH3, MH4, R20, U15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
